Commit message: u

File: urdf/leap_hand.urdf (robot description, URDF)
Before this commit: robot leap_hand, 8 links, 7 joints
Links:
- removed link base_link
- removed link dumay_link
- removed link dumay_link_2
- added link arm_tool_link
- added link dummy_link, mass 0.235; collision mesh filename=../meshes/base_link.stl; visual mesh filename=../meshes/base_link.stl
- added link dummy_link_2, mass 0.235; collision mesh filename=../meshes/palm_lower_left.stl; visual mesh filename=../meshes/palm_lower_left.stl
- added link dummy_link_3
Joints:
- added joint arm_tool_joint: type fixed, parent arm_tool_link, child dummy_link, origin xyz=0.092 -0.071 0.002 rpy=0 -1.5708 -1.5708
- joint dummy_joint: child dumay_link_2 -> dummy_link_2; parent dumay_link -> dummy_link
- joint dummy_joint_2: child base_link -> dummy_link_3; parent dumay_link_2 -> dummy_link_2
- joint joint_1: parent base_link -> dummy_link_3
